File: team tap/team tap.kicad_sch (KiCad schematic)
At the start: 42 parts, among them P1 to console cable, U1 74HC154, U2 74HC244

Commit message: fixed layout and added pcb
Parts:
- C1, C2: value C -> 100nF; footprint (none) -> Capacitor_THT:C_Disc_D4.3mm_W1.9mm_P5.00mm
- C3: value C_Polarized -> 47uF; footprint (none) -> Capacitor_THT:CP_Radial_D5.0mm_P2.50mm
- P1: footprint (none) -> Connector_PinHeader_2.54mm:PinHeader_1x13_P2.54mm_Vertical
- R1, R2, R3, R4, R5, R6: value R -> 4.7k; footprint (none) -> Resistor_THT:R_Axial_DIN0204_L3.6mm_D1.6mm_P2.54mm_Vertical
- R7: footprint (none) -> Resistor_THT:R_Axial_DIN0204_L3.6mm_D1.6mm_P2.54mm_Vertical
- SCK1, SCK2, SCK3, SCK4: footprint (none) -> Connector_Dsub:DSUB-15-HD_Female_Horizontal_P2.29x1.98mm_EdgePinOffset8.35mm_Housed_MountingHolesOffset10.89mm
- U1: footprint (none) -> Package_DIP:DIP-24_W15.24mm
- U2: footprint (none) -> Package_DIP:DIP-20_W7.62mm
Connections:
- net s0: now also SCK2.4; no longer SCK2.14
- net s1: now also SCK2.3; no longer SCK2.13
- net s10: now also SCK4.3; no longer SCK4.13
- net s11: now also SCK1.2; no longer SCK1.12
- net s12: now also SCK4.2; no longer SCK4.12
- net s13: now also SCK1.3; no longer SCK1.13
- net s14: now also SCK1.4; no longer SCK1.14
- net s15: now also SCK4.1; no longer SCK4.11
- net s2: now also SCK2.2; no longer SCK2.12
- net s3: now also SCK2.1; no longer SCK2.11
- net s4: now also SCK3.4; no longer SCK3.14
- net s5: now also SCK3.3; no longer SCK3.13
- net s6: now also SCK3.2; no longer SCK3.12
- net s7: now also SCK1.1; no longer SCK1.11
- net s8: now also SCK3.1; no longer SCK3.11
- net s9: now also SCK4.4; no longer SCK4.14
- net at D2.1 (K): now also SCK1.14; no longer SCK1.4
- net at D17.1 (K): now also SCK3.13; no longer SCK3.3
- net at D21.1 (K): now also SCK4.11; no longer SCK4.1
- net at D22.1 (K): now also SCK4.12; no longer SCK4.2
- net at D23.1 (K): now also SCK4.13; no longer SCK4.3
- net at D24.1 (K): now also SCK4.14; no longer SCK4.4
- net at D14.1 (K): now also SCK3.11; no longer SCK3.1
- net at D18.1 (K): now also SCK3.14; no longer SCK3.4
- net at D11.1 (K): now also SCK2.14; no longer SCK2.4
- net at D8.1 (K): now also SCK2.11; no longer SCK2.1
- net at D9.1 (K): now also SCK2.12; no longer SCK2.2
- net at D10.1 (K): now also SCK2.13; no longer SCK2.3
- net at D5.1 (K): now also SCK1.11; no longer SCK1.1
- net at D15.1 (K): now also SCK3.12; no longer SCK3.2
- net at D4.1 (K): now also SCK1.12; no longer SCK1.2
- net at D3.1 (K): now also SCK1.13; no longer SCK1.3
