File: team tap/team tap.kicad_pcb (KiCad board)
At the start: 2 copper layers, 134.6 x 58.4 mm, 44 parts, among them P1 to console cable, U1 74HC154, U2 74HC244

Commit message: finished all PCBs for this round
Routing:
- net GND: track 567.5 -> 531.8 mm, vias 7 -> 6
- net /s6: track 32.5 -> 30.7 mm
- net /int6: track 182.9 -> 182.1 mm
