File: jaguar spinner top pcb/jaguar controller top pcb.kicad_pcb (KiCad board)
At the start: 2 copper layers, 121 x 45.7 mm, 11 parts, among them J1 Conn_01x13, SW1 Left, SW2 Up, SW3 Down, SW4 Right, SW5 Pause, SW6 Option, SW7 C, SW8 B, SW9 A

Commit message: finished all PCBs for this round
Parts:
- added VR1: PEC11R-4020K-S0024, Evan's misc parts:PEC11R-4XXXK-SXXXX, F.Cu at (58.0, 13.5)
Connections:
- net Net-(J1-Pad12) renamed /encoderB
- net Net-(J1-Pad13) renamed /encoderC
- net Net-(J1-Pad2) renamed /encoderA
Routing:
- net Net-(J1-Pad9): track 45.9 -> 87.6 mm, vias 0 -> 1
- net Net-(J1-Pad8): track 49.6 -> 87.6 mm, vias 0 -> 1
- net Net-(J1-Pad7): track 41.5 -> 71.5 mm, vias 0 -> 1
- net /encoderA: track 145.6 -> 172.2 mm, vias 0 -> 2
- net Net-(J1-Pad6): track 61.4 -> 84.6 mm, vias 0 -> 1
- net /encoderC: track 313.1 -> 333.0 mm
- net /encoderB: track 53.6 -> 72.3 mm
- net Net-(J1-Pad5): track 49.1 -> 64.7 mm, vias 0 -> 1
- net Net-(J1-Pad1): track 124.3 -> 128.6 mm, vias 0 -> 1
- net Net-(J1-Pad11): track 66.4 -> 69.0 mm
