File: jaguar spinner top pcb/jaguar controller top pcb.kicad_sch (KiCad schematic)
At the start: 10 parts, among them J1 Conn_01x13, SW1 Left, SW2 Up, SW3 Down, SW4 Right, SW5 Pause, SW6 Option, SW7 C, SW8 B, SW9 A

Commit message: finished all PCBs for this round
Parts:
- added VR1: PEC11R-4020K-S0024, Evan's misc parts:PEC11R-4XXXK-SXXXX, symbol mouser:PEC11R-4020K-S0024
Connections:
- net encoderC: now reaches J1.13 (Pin_13), SW1.1, SW2.2, SW3.1, SW4.1, SW5.1, SW9.2
- net encoderC: now also VR1.5 (C)
- net encoderA: now reaches J1.2 (Pin_2), SW1.2
- net encoderA: now also VR1.3 (A)
- net encoderB: now reaches J1.12 (Pin_12), SW4.2
- net encoderB: now also VR1.4 (B)
Changed lines of the file:
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@@
     (stroke (width 0) (type default) (color 0 0 0 0))
+  )
+  (label "encoderC" (at 75.565 69.85 180)
+    (effects (font (size 1.27 1.27)) (justify right bottom))
+  )
+  (label "encoderA" (at 85.09 29.845 180)
+    (effects (font (size 1.27 1.27)) (justify right bottom))
+  )
+  (label "encoderB" (at 105.41 24.765 0)
+    (effects (font (size 1.27 1.27)) (justify left bottom))
+  )
+  (label "encoderC" (at 105.41 27.305 0)
+    (effects (font (size 1.27 1.27)) (justify left bottom))
+  )
+  (label "encoderA" (at 89.535 76.2 180)
+    (effects (font (size 1.27 1.27)) (justify right bottom))
+  )
+  (label "encoderB" (at 111.76 68.58 0)
+    (effects (font (size 1.27 1.27)) (justify left bottom))
   )
   (symbol (lib_id "Switch:SW_Push") (at 126.365 95.885 0) (unit 1)
@@
     (pin "1")
     (pin "2")
+  )
+  (symbol (lib_id "mouser:PEC11R-4020K-S0024") (at 85.09 24.765 0) (unit 1)
+    (in_bom yes) (on_board yes) (fields_autoplaced)
+    (property "Reference" "VR1" (id 0) (at 95.25 18.3093 0))
+    (property "Value" "PEC11R-4020K-S0024" (id 1) (at 95.25 21.0844 0))
+    (property "Footprint" "Evan's misc parts:PEC11R-4XXXK-SXXXX" (id 2) (at 101.6 22.225 0)
+      (effects (font (size 1.27 1.27)) (justify left) hide)
+    )
+    (property "Datasheet" "https://www.bourns.com/docs/Product-Datasheets/PEC11R.pdf" (id 3) (at 101.6 24.765 0)
+      (effects (font (size 1.27 1.27)) (justify left) hide)
+    )
+    (property "Description" "Bourns 24 Pulse Incremental Mechanical Rotary Encoder with a 6 mm Knurl Shaft (Not Indexed), Through Hole" (id 4) (at 101.6 27.305 0)
+      (effects (font (size 1.27 1.27)) (justify left) hide)
+    )
+    (property "Height" "" (id 5) (at 101.6 29.845 0)
+      (effects (font (size 1.27 1.27)) (justify left) hide)
+    )
+    (property "Mouser Part Number" "652-PEC11R-4020K-S24" (id 6) (at 101.6 32.385 0)
+      (effects (font (size 1.27 1.27)) (justify left) hide)
+    )
+    (property "Mouser Price/Stock" "https://www.mouser.co.uk/ProductDetail/Bourns/PEC11R-4020K-S0024?qs=Zq5ylnUbLm7F7TcQMKQAfQ%3D%3D" (id 7) (at 101.6 34.925 0)
+      (effects (font (size 1.27 1.27)) (justify left) hide)
+    )
+    (property "Manufacturer_Name" "Bourns" (id 8) (at 101.6 37.465 0)
+      (effects (font (size 1.27 1.27)) (justify left) hide)
+    )
+    (property "Manufacturer_Part_Number" "PEC11R-4020K-S0024" (id 9) (at 101.6 40.005 0)
+      (effects (font (size 1.27 1.27)) (justify left) hide)
+    )
+    (pin "1")
+    (pin "2")
+    (pin "3")
+    (pin "4")
+    (pin "5")
   )
   (symbol (lib_id "Switch:SW_Push") (at 177.8 85.09 0) (unit 1)
@@
       (reference "SW9") (unit 1) (value "A") (footprint "Evan's misc parts:jaguar abc")
     )
-  )
+    (path "/4a49968a-d270-48ca-9d6b-8f64c0d2db7c"
+      (reference "VR1") (unit 1) (value "PEC11R-4020K-S0024") (footprint "Evan's misc parts:PEC11R-4XXXK-SXXXX")
+    )
+  )
